Commit message: Modificación de la matríz 6x6

File: Minichallenge4/urdf/puzzlebot_jetson_ed_urdf.urdf (robot description, URDF)
Before this commit: robot Puzzlebot Jetson-Lidar Ed., 6 links, 5 joints
Links:
- link chassis: geometry collision mesh filename=package://Minichallenge4/models/MCR2_1000_13_Chassis.stl; visual mesh filename=package://Minichallenge4/models/MCR2_1000_13_Chassis.stl
- link lw: geometry collision mesh filename=package://Minichallenge4/models/MCR2_1000_1_1_Wheel_Coupler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; visual mesh filename=package://Minichallenge4/models/MCR2_1000_1_1_Wheel_Coupler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
- link rw: geometry collision mesh filename=package://Minichallenge4//models/MCR2_1000_1_1_Wheel_Couple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; visual mesh filename=package://Minichallenge4/models/MCR2_1000_1_1_Wheel_Coupler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
